Commit message: fix: hip pitch -0.077 to -0.062

File: robots/K1/K1_22dof-ZED.urdf (robot description, URDF)
Before this commit: robot K1, 23 links, 22 joints
Joints:
- joint Left_Hip_Pitch: origin xyz=0 0.096 -0.077 rpy=0 0 0 -> xyz=0 0.096 -0.062 rpy=0 0 0
- joint Right_Hip_Pitch: origin xyz=0 -0.096 -0.077 rpy=0 0 0 -> xyz=0 -0.096 -0.062 rpy=0 0 0

File: robots/K1/K1_22dof.urdf (robot description, URDF)
Before this commit: robot K1, 23 links, 22 joints
Joints:
- joint Left_Hip_Pitch: origin xyz=0 0.096 -0.077 rpy=0 0 0 -> xyz=0 0.096 -0.062 rpy=0 0 0
- joint Right_Hip_Pitch: origin xyz=0 -0.096 -0.077 rpy=0 0 0 -> xyz=0 -0.096 -0.062 rpy=0 0 0

File: robots/K1/K1_locomotion.urdf (robot description, URDF)
Before this commit: robot K1, 23 links, 22 joints
Joints:
- joint Left_Hip_Pitch: origin xyz=0 0.096 -0.077 rpy=0 0 0 -> xyz=0 0.096 -0.062 rpy=0 0 0
- joint Right_Hip_Pitch: origin xyz=0 -0.096 -0.077 rpy=0 0 0 -> xyz=0 -0.096 -0.062 rpy=0 0 0
