Commit message: fix: hip pitch -0.077 to -0.062 (K1, upstream naming)

File: robots/K1/K1_22dof.urdf (robot description, URDF)
Before this commit: robot K1, 25 links, 24 joints
Joints:
- joint left_hip_pitch_joint: origin xyz=0 0.096 -0.077 rpy=0 0 0 -> xyz=0 0.096 -0.062 rpy=0 0 0
- joint right_hip_pitch_joint: origin xyz=0 -0.096 -0.077 rpy=0 0 0 -> xyz=0 -0.096 -0.062 rpy=0 0 0

File: robots/K1/K1_locomotion.urdf (robot description, URDF)
Before this commit: robot K1, 23 links, 22 joints
Joints:
- joint left_hip_pitch_joint: origin xyz=0 0.096 -0.077 rpy=0 0 0 -> xyz=0 0.096 -0.062 rpy=0 0 0
- joint right_hip_pitch_joint: origin xyz=0 -0.096 -0.077 rpy=0 0 0 -> xyz=0 -0.096 -0.062 rpy=0 0 0
